File: WSC6502.kicad_pcb (KiCad board)
At the start: 2 copper layers, 139.7 x 157 mm, 26 parts, among them IC1 W65C02S6TPG-14 CPU, IC2 AT28C256-15PU ROM, IC3 AS6C62256-55PCN SRAM, IC4 W65C22S6TPG-14 I/O, SW1 Reset, SW2 , SW3 , SW5 , SW6 , U1 74HC00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

Commit message: Add files via upload
Parts:
- renumbered SW5 to SW4
Connections:
- Y1 pad 14: +5V -> GND
- Y1 pad 7: GND -> +5V
