File: WSC6502.kicad_pcb (KiCad board)
At the start: 2 copper layers, 139.7 x 157 mm, 26 parts, among them IC1 W65C02S6TPG-14 CPU, IC2 AT28C256-15PU ROM, IC3 AS6C62256-55PCN SRAM, IC4 W65C22S6TPG-14 I/O, SW1 Reset, SW2 , SW3 , SW4 , SW5 , SW6 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

Commit message: Add files via upload
Parts:
- added J1: +5V, Connector_PinHeader_2.54mm:PinHeader_1x02_P2.54mm_Vertical, F.Cu at (50.0, 159.5)
- added J2: +5V, Connector_BarrelJack:BarrelJack_Horizontal, F.Cu at (40.3, 159.5)
- added REF**: OSHW-Logo2_9.8x8mm_SilkScreen, Symbol:OSHW-Logo2_9.8x8mm_SilkScreen, B.Cu at (145.4, 165.5)
- added REF**: , Symbol:Polarity_Center_Positive_6mm_SilkScreen, F.Cu at (42.2, 148.4)
Other:
- board text added: "+"
- board text added: "Circuit design by Ben Eater https://eater.net/6502 PCB design by RSB http://www.thebrunonet.com"

Commit message: Add files via upload
Parts:
- DS1: footprint Display:HY1602E -> Display:WC1602A
- moved RV1 58.9 mm to (50.0, 83.9), turned to 0 degrees
- moved DS1 43.9 mm to (65.2, 94.0)
- moved C3 9.78 mm to (138.0, 81.5), turned to 0 degrees
- moved C2 0.29 mm to (112.6, 66.4)
Routing:
- net Net-(DS1-Pad4): track 54.9 -> 101.6 mm
- net Net-(DS1-Pad9): track 31.6 -> 78.0 mm
- net Net-(DS1-Pad5): track 50.6 -> 96.8 mm
- net Net-(DS1-Pad6): track 45.9 -> 92.1 mm
- net Net-(DS1-Pad7): track 41.2 -> 87.4 mm
- net Net-(DS1-Pad8): track 36.5 -> 82.7 mm
- net Net-(DS1-Pad10): track 27.8 -> 73.3 mm
- net Net-(DS1-Pad11): track 24.2 -> 68.6 mm
- net Net-(DS1-Pad12): track 22.3 -> 63.9 mm
- net Net-(DS1-Pad13): track 19.2 -> 59.2 mm
- net Net-(DS1-Pad14): track 17.8 -> 54.2 mm
- net Net-(DS1-Pad3): track 10.3 -> 21.2 mm
- net /a14: track 185.9 -> 184.0 mm

Commit message: Add files via upload
Parts:
- removed the REF** at (42.2, 148.4)
- J2: value +5V -> +5V in
- moved R6 56.4 mm to (60.6, 148.2), turned to 0 degrees
- moved J1 36.1 mm to (34.2, 127.1)
- moved SW6 31.2 mm to (107.7, 143.0)
- moved R5 30.2 mm to (60.6, 158.9)
- moved SW5 27.7 mm to (79.2, 143.0)
- moved SW3 24.1 mm to (100.0, 138.6)
- moved SW2 23.8 mm to (136.0, 152.0)
- moved R7 16.6 mm to (60.6, 155.3), turned to 0 degrees
- moved R3 15.8 mm to (128.4, 159.5), turned to 0 degrees
- moved R4 12.7 mm to (60.6, 151.8), turned to 0 degrees
- moved SW4 7.87 mm to (99.9, 156.3)
Connections:
- J2 pad 3: (no net) -> GND
Routing:
- net Net-(IC4-Pad5): track 149.5 -> 184.5 mm
- net Net-(IC4-Pad4): track 167.7 -> 188.4 mm, vias 0 -> 1
- net Net-(IC4-Pad6): track 227.2 -> 208.9 mm
- net Net-(IC4-Pad2): track 153.7 -> 146.7 mm, vias 0 -> 1
- net Net-(IC4-Pad3): track 186.8 -> 190.5 mm

Commit message: Add files via upload
Parts:
- moved R1 33.1 mm to (75.2, 64.8), turned to 180 degrees
- moved R2 25.1 mm to (35.3, 48.9), turned to 0 degrees
- moved RV1 18.0 mm to (67.8, 81.1), turned to 90 degrees
Routing:
- net Net-(IC1-Pad2): track 37.4 -> 3.80 mm
- net Net-(IC1-Pad37): track 171.4 -> 153.7 mm
- net Net-(IC2-Pad20): track 76.7 -> 67.4 mm
- net Net-(IC4-Pad23): track 124.6 -> 116.7 mm
- net /a15: track 59.9 -> 53.1 mm
- net Net-(DS1-Pad3): track 21.2 -> 15.8 mm
- net Net-(C1-Pad1): track 217.6 -> 221.3 mm
- net /a14: track 184.0 -> 180.9 mm
- net Net-(IC3-Pad20): track 122.0 -> 120.0 mm
- net Net-(IC1-Pad4): track 160.8 -> 159.0 mm
- net /a3: track 160.7 -> 159.4 mm
- net /a4: track 133.0 -> 131.7 mm
- net /a5: track 133.5 -> 132.6 mm

Commit message: Add files via upload
Parts:
- added D1: , LED_THT:LED_D3.0mm, F.Cu at (157.1, 44.3)
- added D2: , LED_THT:LED_D3.0mm, F.Cu at (157.1, 48.9)
- added D3: , LED_THT:LED_D3.0mm, F.Cu at (157.1, 53.5)
- added D4: , LED_THT:LED_D3.0mm, F.Cu at (157.1, 58.0)
- added D5: , LED_THT:LED_D3.0mm, F.Cu at (157.1, 62.6)
- added D6: , LED_THT:LED_D3.0mm, F.Cu at (157.1, 67.2)
- added D7: , LED_THT:LED_D3.0mm, F.Cu at (157.1, 71.8)
- added D8: , LED_THT:LED_D3.0mm, F.Cu at (157.1, 76.4)
- added J3: Address Bus, Connector_PinHeader_2.54mm:PinHeader_2x16_P2.54mm_Vertical, B.Cu at (53.1, 72.3)
- added J4: Data Bus, Connector_PinHeader_2.54mm:PinHeader_2x08_P2.54mm_Vertical, B.Cu at (96.1, 72.3)
- added RN1: 220R, Resistor_THT:R_Array_SIP9, F.Cu at (164.8, 49.0)
- J2: value +5V in -> +5V
- moved R1 86.1 mm to (157.6, 39.6), turned to 90 degrees
- moved C2 42.7 mm to (125.4, 25.7), turned to 0 degrees
- moved J1 16.5 mm to (40.5, 142.4), turned to 270 degrees
- moved RV1 15.0 mm to (54.2, 87.5)
- moved J2 5.15 mm to (42.7, 155.0)
- moved C1 2.26 mm to (37.0, 74.2)
Connections:
- net Net-(DS1-Pad10) renamed /DS1-D3
- net Net-(DS1-Pad11) renamed /DS1-D4
- net Net-(DS1-Pad12) renamed /DS1-D5
- net Net-(DS1-Pad13) renamed /DS1-D6
- net Net-(DS1-Pad14) renamed /DS1-D7
- net Net-(DS1-Pad3) renamed /DS1-V0
- net Net-(DS1-Pad4) renamed /DS1-RS
- net Net-(DS1-Pad5) renamed /DS1-R~W
- net Net-(DS1-Pad6) renamed /DS1-Ena
- net Net-(DS1-Pad7) renamed /DS1-D0
- net Net-(DS1-Pad8) renamed /DS1-D1
- net Net-(DS1-Pad9) renamed /DS1-D2
- J2 pad 3: GND -> (no net)
- RV1 pad 3: Net-(RV1-Pad3) -> +5V
Routing:
- net /d3: track 110.5 -> 174.5 mm, vias 2 -> 4
- net /a14: track 180.9 -> 241.7 mm, vias 2 -> 3
- net /a15: track 53.1 -> 111.9 mm, vias 1 -> 7
- net /d4: track 109.0 -> 163.8 mm, vias 2 -> 4
- net /a12: track 75.6 -> 129.9 mm, vias 0 -> 1
- net /d5: track 108.3 -> 158.2 mm, vias 2 -> 4
- net /d6: track 107.4 -> 155.4 mm
- net /d1: track 131.9 -> 178.9 mm, vias 1 -> 4
- net /d2: track 131.2 -> 177.7 mm, vias 1 -> 3
- net /d0: track 129.6 -> 175.4 mm, vias 1 -> 3
- net /d7: track 106.5 -> 150.1 mm
- net /a13: track 111.5 -> 148.2 mm, vias 0 -> 1
- net /a6: track 134.2 -> 162.3 mm
- net /a2: track 158.7 -> 186.5 mm
- net /a0: track 157.6 -> 185.3 mm
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Other:
- board size 139.7 x 157 mm -> 145.6 x 157 mm
- board text added: "0 1 2 4 8 16 32 64"
- board text added: "5 v"
- board text added: "Address Bus"
- board text added: "Data Bus"
- board text added: "G N D"
- board text added: "Rev 1.0"
- board text added: "a 0"
- board text added: "a 1 5"
- board text added: "d 0"
- board text added: "d 7"

Commit message: Add files via upload
Parts:
- added JP1: Jumper_2_Bridged, Connector_PinSocket_2.54mm:PinSocket_1x02_P2.54mm_Vertical, F.Cu at (72.1, 56.7)
- moved C1 11.1 mm to (44.4, 65.8), turned to 0 degrees
Connections:
- Y1 pad 8: Net-(IC1-Pad37) -> Net-(JP1-Pad1)
Routing:
- net Net-(JP1-Pad1): track 0.00 -> 6.90 mm
- net /d1: track 178.9 -> 175.2 mm
- net Net-(C1-Pad1): track 220.7 -> 223.4 mm
- net Net-(IC3-Pad20): track 117.4 -> 117.9 mm
Other:
- board text added: "256k RAM"
- board text added: "32K ROM"
- board text added: "6502 CPU"
- board text added: "CLK In"
- board text added: "I/O Controller"
- board text added: "Reset"
- board text added: "XTAL Out"

Commit message: Add files via upload
Parts:
- added J5: R~W TP, Connector_PinHeader_2.54mm:PinHeader_1x01_P2.54mm_Vertical, F.Cu at (45.5, 24.4)
- added J6: , Connector_PinHeader_2.54mm:PinHeader_1x01_P2.54mm_Vertical, F.Cu at (161.5, 24.4)
- JP1: value Jumper_2_Bridged -> Clock INT / EXT; footprint Connector_PinSocket_2.54mm:PinSocket_1x02_P2.54mm_Vertical -> Connector_PinSocket_2.54mm:PinSocket_1x03_P2.54mm_Vertical
- moved JP1 0.57 mm to (72.1, 56.1)
Connections:
- net Net-(IC1-Pad34) renamed /R~W
Routing:
- net /R~W: track 130.6 -> 137.8 mm
- net Net-(IC4-Pad5): track 177.8 -> 181.8 mm
- net Net-(IC4-Pad6): track 207.0 -> 210.2 mm
- net /a8: track 74.0 -> 72.3 mm
- net Net-(IC1-Pad37): track 151.7 -> 153.2 mm
- net Net-(IC4-Pad3): track 190.5 -> 191.5 mm
- net /a9: track 70.2 -> 69.1 mm
- net Net-(IC3-Pad20): track 117.9 -> 118.5 mm
Other:
- board text added: "CLK TP"
- board text added: "GND"
- board text added: "R/~W"

Commit message: Add files via upload
Parts:
- moved R1 123.6 mm to (39.1, 74.7), turned to 0 degrees
- moved D8 84.5 mm to (74.4, 93.7), turned to 90 degrees
- moved D7 81.1 mm to (79.0, 93.7), turned to 90 degrees
- moved D6 78.2 mm to (83.6, 93.7), turned to 90 degrees
- moved D5 75.7 mm to (88.1, 93.7), turned to 90 degrees
- moved D4 73.6 mm to (92.7, 93.7), turned to 90 degrees
- moved RN1 72.3 mm to (101.3, 83.8), turned to 180 degrees
- moved D3 72.1 mm to (97.3, 93.7), turned to 90 degrees
- moved D2 71.2 mm to (101.9, 93.7), turned to 90 degrees
- moved D1 70.8 mm to (106.4, 93.7), turned to 90 degrees
- moved RV1 11.4 mm to (48.1, 97.2)
- moved DS1 11.4 mm to (59.2, 103.6)
- moved SW2 9.75 mm to (128.8, 158.5)
- moved R3 9.75 mm to (121.2, 166.0)
- moved R4 9.75 mm to (53.3, 158.3)
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Connections:
- net Net-(C1-Pad1) renamed /~Reset
- D1 pad 1: /d0 -> DS1-D0
- D2 pad 1: /d1 -> DS1-D1
- D3 pad 1: /d2 -> DS1-D2
- D4 pad 1: /d3 -> DS1-D3
- D5 pad 1: /d4 -> DS1-D4
- D6 pad 1: /d5 -> DS1-D5
- D7 pad 1: /d6 -> DS1-D6
- D8 pad 1: /d7 -> DS1-D7
- DS1 pad 10: /DS1-D3 -> DS1-D3
- DS1 pad 11: /DS1-D4 -> DS1-D4
- DS1 pad 12: /DS1-D5 -> DS1-D5
- DS1 pad 13: /DS1-D6 -> DS1-D6
- DS1 pad 14: /DS1-D7 -> DS1-D7
- DS1 pad 7: /DS1-D0 -> DS1-D0
- DS1 pad 8: /DS1-D1 -> DS1-D1
- DS1 pad 9: /DS1-D2 -> DS1-D2
- IC4 pad 10: /DS1-D0 -> DS1-D0
- IC4 pad 11: /DS1-D1 -> DS1-D1
- IC4 pad 12: /DS1-D2 -> DS1-D2
- IC4 pad 13: /DS1-D3 -> DS1-D3
- IC4 pad 14: /DS1-D4 -> DS1-D4
- IC4 pad 15: /DS1-D5 -> DS1-D5
- IC4 pad 16: /DS1-D6 -> DS1-D6
- IC4 pad 17: /DS1-D7 -> DS1-D7
Routing:
- net DS1-D0: track 0.00 -> 145.7 mm
- net DS1-D1: track 0.00 -> 136.6 mm
- net DS1-D2: track 0.00 -> 130.7 mm
- net DS1-D3: track 0.00 -> 126.5 mm
- net DS1-D4: track 0.00 -> 122.0 mm
- net DS1-D5: track 0.00 -> 117.4 mm
- net DS1-D6: track 0.00 -> 112.9 mm
- net DS1-D7: track 0.00 -> 108.6 mm
- net /DS1-D0: track 87.4 -> 0.00 mm
- net /DS1-D1: track 82.7 -> 0.00 mm
- net /DS1-D2: track 78.0 -> 0.00 mm
- net /DS1-D3: track 73.3 -> 0.00 mm
- net /DS1-D4: track 68.6 -> 0.00 mm
- net /DS1-D5: track 63.9 -> 0.00 mm
- net /DS1-D6: track 59.2 -> 0.00 mm
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Other:
- board text added: "0"
- board text added: "1"
- board text added: "16"
- board text added: "2"
- board text added: "32"
- board text added: "4"
- board text added: "64"
- board text added: "8"
- board text added: "B0"
- board text added: "B1"
- board text added: "B2"
- board text added: "B3"
- board text added: "B4"
- board text added: "B5"
- board text added: "B6"
- board text added: "B7"
- board text added: "Port"
- board text added: "Rev 1.5"
- board text removed: "0 1 2 4 8 16 32 64"
- board text removed: "Rev 1.0"
