File: WSC6502.kicad_pcb (KiCad board)
At the start: 2 copper layers, 145.6 x 157 mm, 43 parts, among them IC1 W65C02S6TPG-14 CPU, IC2 AT28C256-15PU ROM, IC3 AS6C62256-55PCN SRAM, IC4 W65C22S6TPG-14 I/O, J1 +5V, J2 +5V, J3 Address Bus, J4 Data Bus, J5 R~W TP, J6 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

Commit message: Add files via upload
Parts:
- J5: value R~W TP -> R~W~ TP
- moved R3 20.6 mm to (140.4, 158.5), turned to 180 degrees
- moved R4 5.31 mm to (53.8, 153.1)
- moved R5 5.31 mm to (53.8, 160.2)
- moved R6 5.31 mm to (53.8, 149.5)
- moved R7 5.31 mm to (53.8, 156.6)
- moved C2 0.92 mm to (125.3, 26.6)
- moved U1 0.08 mm to (32.7, 60.5)
Connections:
- net DS1-D0 renamed PB0-DS1-D0
- net DS1-D1 renamed PB1-DS1-D1
- net DS1-D2 renamed PB2-DS1-D2
- net DS1-D3 renamed PB3-DS1-D3
- net DS1-D4 renamed PB4-DS1-D4
- net DS1-D5 renamed PB5-DS1-D5
- net DS1-D6 renamed PB6-DS1-D6
- net DS1-D7 renamed PB7-DS1-D7
Routing:
- net Net-(IC1-Pad4): track 157.8 -> 161.7 mm
- net Net-(IC4-Pad6): track 214.9 -> 218.6 mm
- net Net-(IC4-Pad2): track 152.7 -> 149.2 mm
- net Net-(IC4-Pad5): track 186.1 -> 183.7 mm
- net Net-(IC4-Pad3): track 196.9 -> 199.3 mm
- net /a13: track 148.2 -> 146.1 mm
- net PB2-DS1-D2: track 130.7 -> 129.1 mm
- net Net-(IC3-Pad20): track 118.5 -> 116.9 mm
- net /a14: track 241.7 -> 243.2 mm
- net PB3-DS1-D3: track 126.5 -> 125.5 mm
- net PB1-DS1-D1: track 136.6 -> 135.6 mm
- net /a15: track 111.9 -> 111.0 mm
- net /a0: track 185.3 -> 186.1 mm
- net Net-(JP1-Pad1): track 7.39 -> 6.76 mm
- net Net-(IC4-Pad4): track 193.8 -> 193.3 mm
Other:
- board text added: "R/~W~"
- board text removed: "R/~W"

Commit message: Add files via upload
Connections:
- net Net-(IC1-Pad37) renamed /CLK
- net Net-(IC1-Pad4) renamed /~IRQ~
- net Net-(IC3-Pad20) renamed /~CE~
- net Net-(IC4-Pad23) renamed /~CS2~
Routing:
- net PB3-DS1-D3: track 125.5 -> 126.1 mm
- net PB0-DS1-D0: track 146.1 -> 145.5 mm
- net /a0: track 186.1 -> 185.6 mm

Commit message: Add files via upload
Connections:
- IC1 pad 39: Net-(IC1-Pad39) -> +5V
Routing:
- net /d1: track 171.3 -> 170.6 mm

Commit message: Add files via upload
Connections:
- IC1 pad 36: Net-(IC1-Pad36) -> +5V
- IC1 pad 39: +5V -> Net-(IC1-Pad39)
Routing:
- net /a1: track 184.9 -> 182.0 mm, vias 1 -> 3
- net /a0: track 185.6 -> 187.2 mm, vias 1 -> 3
- net /CLK: track 152.7 -> 153.3 mm, vias 1 -> 2

Commit message: Add files via upload
Routing:
- net /CLK: track 153.3 -> 153.6 mm, vias 2 -> 1
Changed lines of the file:
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@@
     (thickness 1.6)
     (drawings 70)
-    (tracks 1125)
+    (tracks 1123)
     (zones 0)
     (modules 43)
@@
   (segment (start 72.136 58.674) (end 68.326 54.864) (width 0.25) (layer F.Cu) (net 70))
   (segment (start 68.326 54.864) (end 65.914 54.864) (width 0.25) (layer F.Cu) (net 70))
-  (via (at 42.3672 32.258) (size 0.8) (drill 0.4) (layers F.Cu B.Cu) (net 70))
-  (segment (start 40.3606 30.3085) (end 42.3101 32.258) (width 0.25) (layer B.Cu) (net 70))
-  (segment (start 42.3101 32.258) (end 42.3672 32.258) (width 0.25) (layer B.Cu) (net 70))
   (segment (start 40.3606 29.9085) (end 40.3606 30.3085) (width 0.25) (layer B.Cu) (net 70))
   (via (at 45.211998 35.814) (size 0.8) (drill 0.4) (layers F.Cu B.Cu) (net 70))
@@
   (segment (start 44.303984 36.722014) (end 44.811999 36.213999) (width 0.25) (layer B.Cu) (net 70))
   (segment (start 44.811999 36.213999) (end 45.211998 35.814) (width 0.25) (layer B.Cu) (net 70))
-  (segment (start 44.811999 35.414001) (end 45.211998 35.814) (width 0.25) (layer F.Cu) (net 70))
-  (segment (start 42.3672 32.969202) (end 44.811999 35.414001) (width 0.25) (layer F.Cu) (net 70))
-  (segment (start 42.3672 32.258) (end 42.3672 32.969202) (width 0.25) (layer F.Cu) (net 70))
+  (segment (start 40.3606 30.3085) (end 40.3606 29.9085) (width 0.25) (layer F.Cu) (net 70))
+  (segment (start 42.3672 32.3151) (end 40.3606 30.3085) (width 0.25) (layer F.Cu) (net 70))
+  (segment (start 45.211998 35.814) (end 42.3672 32.969202) (width 0.25) (layer F.Cu) (net 70))
+  (segment (start 42.3672 32.969202) (end 42.3672 32.3151) (width 0.25) (layer F.Cu) (net 70))
   (via (at 117.5385 63.119) (size 0.8) (drill 0.4) (layers F.Cu B.Cu) (net 71))
   (segment (start 47.8536 53.2955) (end 47.8536 52.8955) (width 0.25) (layer F.Cu) (net 71))
